File: Hardware/HybrideNixieClock.brd (EAGLE design)
At the start: 81.5 x 52.5 mm, 78 parts, among them IC2 ESP-12E/F, Q1 mmbt2222, Q2 mmbt2222, SW1 KMR2, SW2 KMR2, T1 MJE340, T2 MJE340, U1 LM3481MM, U2 AP2112-3.3, U3 MCP73831T-2ACI/OT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

Commit message: Final V1 Hardware
Parts:
- added CHG1: ORANGE, microbuilder:CHIPLED_0805_NOOUTLINE
- added R26: 1K, microbuilder:0603-NO
- C16, C17, C18, C19: value 22pF -> 47uF
- R18, R19, R21, R22: value 1K -> 3.9K
- R23: value 1K -> 270R
- moved U4 1.58 mm to (60.0, 43.0)
- moved R15 1.50 mm to (77.0, 42.5)
Connections:
- new net N$30: CHG1.A, R26.1
- net 3.3V: now also R26.2
- net GND: now also CHG1.C
Routing:
- net 3.3V: track 269.6 -> 276.7 mm
- net N$30: track 0.00 -> 2.08 mm
- net ISENSE: track 13.7 -> 11.7 mm
- net N$6: track 11.1 -> 9.48 mm
- net N$11: track 22.8 -> 24.3 mm
- net FB: track 39.1 -> 40.3 mm
- net N$19: track 8.55 -> 7.58 mm
Other:
- board text added: "Charge"
- board text added: "Ext. Supply"
- board text added: "Gyro Powerd"
- board text added: "IN 9 Nixie Tubes"
- board text added: "MJE340"
- board text added: "ON"
- board text added: "Onboard Supply"
- board text removed: "External Supply"
- board text removed: "Gyro Inside"
- board text removed: "On-Board Supply"
